Commit message: human_model package copied to project

File: urdf/human.urdf.xacro (robot description, xacro)
@@ -25,9 +25,9 @@
 	<!--Link base (1)-->
 	<link name="Hip_mocap">
-        <inertial>
-            <mass value="5.696"/>
-            <origin xyz="0 0 0" rpy="0 0 0" />
-            <inertia ixx="0" iyy="0" izz="0" ixy="0" ixz="0" iyz="0"/>
-        </inertial>
+        <!-- <inertial>
+            <mass value="0"/>
+            <origin xyz="0 0 0" rpy="0 0 0" />
+            <inertia ixx="0" iyy="0" izz="0" ixy="0" ixz="0" iyz="0"/>
+        </inertial> -->
     </link>
 	<link name="hip">
